File: SD2IEC.kicad_pcb (KiCad board)
At the start: 2 copper layers, 64 x 50 mm, 47 parts, among them J1 AVR-ISP-6, J2 5VDC IN, J3 SD_Card, J4 IEC (DIN6), J5 IEC (DIN6), J8 IEC_ALT1, J9 IEC_ALT2, Q1 AO3400A, Q2 AO3400A, Q3 AO3400A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

Commit message: Cleanup
Parts:
- added G***: LOGO, DTLib:Logo, F.Cu at (121.4, 119.8)
- added H1: MountingHole_Pad, MountingHole:MountingHole_2.2mm_M2_DIN965_Pad, F.Cu at (86.3, 126.2)
- added H2: MountingHole_Pad, MountingHole:MountingHole_2.2mm_M2_DIN965_Pad, F.Cu at (145.3, 126.2)
- added H3: MountingHole_Pad, MountingHole:MountingHole_2.2mm_M2_DIN965_Pad, F.Cu at (86.3, 81.2)
- added H4: MountingHole_Pad, MountingHole:MountingHole_2.2mm_M2_DIN965_Pad, F.Cu at (145.3, 81.2)
- moved D2 29.4 mm to (139.7, 126.4), turned to 180 degrees
- moved D3 28.0 mm to (134.6, 126.4), turned to 180 degrees
- moved SW4 12.6 mm to (106.7, 119.3)
- moved SW1 7.95 mm to (99.0, 85.0), turned to 180 degrees
- moved J5 0.76 mm to (147.8, 93.4)
- moved J2 0.51 mm to (84.3, 103.7)
Connections:
- D2 pad 2: Net-(D2-Pad2) -> /DIRTY_LED
- D3 pad 2: Net-(D3-Pad2) -> /BUSY_LED
- R16 pad 1: Net-(D3-Pad2) -> /BUSY_LED
- R16 pad 2: /BUSY_LED -> /BUSY
- R17 pad 1: Net-(D2-Pad2) -> /DIRTY_LED
- R17 pad 2: /DIRTY_LED -> /DIRTY
- U1 pad 19: /BUSY_LED -> /BUSY
- U1 pad 20: /DIRTY_LED -> /DIRTY
Routing:
- net GND: track 57.5 -> 385.1 mm, vias 22 -> 28
- net /PREV: track 0.00 -> 55.6 mm
- net /NEXT: track 0.00 -> 41.8 mm
- net /IEC10_11: track 0.00 -> 32.8 mm, vias 0 -> 1
- net /IEC8_9: track 0.00 -> 32.3 mm, vias 0 -> 1
- net Net-(J1-Pad5): track 39.2 -> 70.2 mm, vias 2 -> 3
- net /DIRTY_LED: track 3.19 -> 30.2 mm
- net /BUSY_LED: track 3.51 -> 27.9 mm
- net +3.3V: track 136.5 -> 120.3 mm, vias 1 -> 2
- net /~{WRITE_PROTECT}: track 20.8 -> 30.3 mm
- net /~{IEC_RESET}: track 72.2 -> 66.7 mm
- net unconnected-(J2-Pad5): track 8.96 -> 14.3 mm
- net unconnected-(J2-Pad4): track 9.03 -> 14.2 mm
- net unconnected-(J2-Pad3): track 9.11 -> 13.8 mm
- net /SCK: track 33.7 -> 38.4 mm
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Other:
- outline, holes or cut-outs redrawn
- board text added: "DEVICE NUMBER"
- board text added: "NEXT"
- board text added: "PREV"
- board text added: "RESET"
- board text added: "SD2IEC RevA 2022 Dominic Thibodeau / dev@hotkeysoft.net https://github.com/hotkeysoft/sd2iec-kicad"
