File: SD2IEC.kicad_sch (KiCad schematic)
At the start: 34 parts, among them J1 AVR-ISP-6, J2 5VDC IN, J3 SD_Card, J4 IEC (DIN6), J5 IEC (DIN6), J6 SERIAL, J7 I2C, J8 IEC_ALT1, J9 IEC_ALT2, SW1 IEC_SEL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

Commit message: Begin routing
Parts:
- removed J6: SERIAL, Connector_PinHeader_2.54mm:PinHeader_1x03_P2.54mm_Vertical, symbol Connector_Generic:Conn_01x03
- removed J7: I2C, Connector_PinHeader_2.54mm:PinHeader_1x04_P2.54mm_Vertical, symbol Connector_Generic:Conn_01x04
Connections:
- net INTRQ: no longer names the net of U1.25 (PC6)
- net RXD: no longer names the net of U1.9 (PD0)
- net SCL: no longer names the net of U1.23 (PC4)
- net SDA: no longer names the net of U1.24 (PC5)
- net TXD: no longer names the net of U1.10 (PD1)
- no-connect marks 13 -> 16
Other:
- moved on the sheet: D2, D3, R16, R17, SW2, SW3

Commit message: Cleanup
Parts:
- added H1, H2, H3, H4: MountingHole_Pad, MountingHole:MountingHole_2.2mm_M2_DIN965_Pad, symbol Mechanical:MountingHole_Pad
Connections:
- net BUSY_LED: now also D3.2 (A), R16.1; no longer R16.2, U1.19 (PC0)
- net DIRTY_LED: now also D2.2 (A), R17.1; no longer R17.2, U1.20 (PC1)
- net GND: now also H1.1, H2.1, H3.1, H4.1
- new net BUSY: R16.2, U1.19 (PC0)
- new net DIRTY: R17.2, U1.20 (PC1)
Changed lines of the file:
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@@
   (title_block
     (title "SD2IEC")
-    (date "2021-07-01")
+    (date "2022-09-18")
     (rev "A")
     (comment 1 "R2 R3 Can be omitted")
@@
   (junction (at 190.5 29.21) (diameter 0) (color 0 0 0 0)
   )
+  (junction (at 254 156.21) (diameter 0) (color 0 0 0 0)
+  )
   (junction (at 207.01 29.21) (diameter 0) (color 0 0 0 0)
   )
@@
   )
   (junction (at 45.72 182.88) (diameter 0) (color 0 0 0 0)
+  )
+  (junction (at 251.46 156.21) (diameter 0) (color 0 0 0 0)
+  )
+  (junction (at 248.92 156.21) (diameter 0) (color 0 0 0 0)
   )
   (junction (at 143.51 179.07) (diameter 0) (color 0 0 0 0)
@@
     (stroke (width 0) (type default) (color 0 0 0 0))
   )
+  (wire (pts (xy 254 153.67) (xy 254 156.21))
+    (stroke (width 0) (type default) (color 0 0 0 0))
+  )
   (wire (pts (xy 255.27 77.47) (xy 255.27 62.23))
     (stroke (width 0) (type default) (color 0 0 0 0))
@@
     (stroke (width 0) (type default) (color 0 0 0 0))
   )
+  (wire (pts (xy 254 156.21) (xy 259.08 156.21))
+    (stroke (width 0) (type default) (color 0 0 0 0))
+  )
   (wire (pts (xy 191.77 59.69) (xy 191.77 66.04))
     (stroke (width 0) (type default) (color 0 0 0 0))
@@
     (stroke (width 0) (type default) (color 0 0 0 0))
   )
+  (wire (pts (xy 251.46 156.21) (xy 254 156.21))
+    (stroke (width 0) (type default) (color 0 0 0 0))
+  )
   (wire (pts (xy 181.61 31.75) (xy 181.61 29.21))
     (stroke (width 0) (type default) (color 0 0 0 0))
@@
     (stroke (width 0) (type default) (color 0 0 0 0))
   )
+  (wire (pts (xy 251.46 156.21) (xy 251.46 158.75))
+    (stroke (width 0) (type default) (color 0 0 0 0))
+  )
   (wire (pts (xy 100.33 95.25) (xy 100.33 85.09))
     (stroke (width 0) (type default) (color 0 0 0 0))
@@
     (stroke (width 0) (type default) (color 0 0 0 0))
   )
+  (wire (pts (xy 243.84 156.21) (xy 248.92 156.21))
+    (stroke (width 0) (type default) (color 0 0 0 0))
+  )
   (wire (pts (xy 83.82 97.79) (xy 93.98 97.79))
     (stroke (width 0) (type default) (color 0 0 0 0))
@@
     (stroke (width 0) (type default) (color 0 0 0 0))
   )
+  (wire (pts (xy 259.08 153.67) (xy 259.08 156.21))
+    (stroke (width 0) (type default) (color 0 0 0 0))
+  )
   (wire (pts (xy 189.23 59.69) (xy 189.23 62.23))
     (stroke (width 0) (type default) (color 0 0 0 0))
@@
     (stroke (width 0) (type default) (color 0 0 0 0))
   )
+  (wire (pts (xy 248.92 153.67) (xy 248.92 156.21))
+    (stroke (width 0) (type default) (color 0 0 0 0))
+  )
   (wire (pts (xy 45.72 100.33) (xy 45.72 97.79))
     (stroke (width 0) (type default) (color 0 0 0 0))
@@
     (stroke (width 0) (type default) (color 0 0 0 0))
   )
+  (wire (pts (xy 243.84 153.67) (xy 243.84 156.21))
+    (stroke (width 0) (type default) (color 0 0 0 0))
+  )
   (wire (pts (xy 215.9 118.11) (xy 215.9 166.37))
     (stroke (width 0) (type default) (color 0 0 0 0))
@@
   )
   (wire (pts (xy 33.02 86.36) (xy 40.64 86.36))
+    (stroke (width 0) (type default) (color 0 0 0 0))
+  )
+  (wire (pts (xy 248.92 156.21) (xy 251.46 156.21))
     (stroke (width 0) (type default) (color 0 0 0 0))
   )
@@
     (effects (font (size 1.27 1.27)) (justify left bottom))
   )
+  (label "DIRTY_LED" (at 118.11 130.81 0)
+    (effects (font (size 1.27 1.27)) (justify left bottom))
+  )
   (label "SCK" (at 95.25 123.19 0)
     (effects (font (size 1.27 1.27)) (justify left bottom))
@@
     (effects (font (size 1.27 1.27)) (justify right bottom))
   )
-  (label "BUSY_LED" (at 87.63 128.27 0)
+  (label "BUSY" (at 87.63 128.27 0)
     (effects (font (size 1.27 1.27)) (justify left bottom))
   )
@@
     (effects (font (size 1.27 1.27)) (justify left bottom))
   )
-  (label "DIRTY_LED" (at 87.63 130.81 0)
+  (label "DIRTY" (at 87.63 130.81 0)
     (effects (font (size 1.27 1.27)) (justify left bottom))
   )
@@
   (label "IEC_ATN" (at 158.75 66.04 180)
     (effects (font (size 1.27 1.27)) (justify right bottom))
+  )
+  (label "BUSY_LED" (at 118.11 128.27 0)
+    (effects (font (size 1.27 1.27)) (justify left bottom))
   )
   (symbol (lib_id "MCU_Microchip_ATmega:ATmega1284P-A") (at 68.58 125.73 0) (unit 1)
@@
     (pin "2")
   )
+  (symbol (lib_id "Mechanical:MountingHole_Pad") (at 254 151.13 0) (unit 1)
+    (in_bom yes) (on_board yes)
+    (property "Reference" "H3" (id 0) (at 252.73 146.05 0)
+      (effects (font (size 1.27 1.27)) (justify left))
+    )
+    (property "Value" "MountingHole_Pad" (id 1) (at 256.54 151.5622 0)
+      (effects (font (size 1.27 1.27)) (justify left) hide)
+    )
+    (property "Footprint" "MountingHole:MountingHole_2.2mm_M2_DIN965_Pad" (id 2) (at 254 151.13 0)
+      (effects (font (size 1.27 1.27)) hide)
+    )
+    (property "Datasheet" "~" (id 3) (at 254 151.13 0)
+      (effects (font (size 1.27 1.27)) hide)
+    )
+    (pin "1")
+  )
+  (symbol (lib_id "Mechanical:MountingHole_Pad") (at 243.84 151.13 0) (unit 1)
+    (in_bom yes) (on_board yes)
+    (property "Reference" "H1" (id 0) (at 242.57 146.05 0)
+      (effects (font (size 1.27 1.27)) (justify left))
+    )
+    (property "Value" "MountingHole_Pad" (id 1) (at 246.38 151.5622 0)
+      (effects (font (size 1.27 1.27)) (justify left) hide)
+    )
+    (property "Footprint" "MountingHole:MountingHole_2.2mm_M2_DIN965_Pad" (id 2) (at 243.84 151.13 0)
+      (effects (font (size 1.27 1.27)) hide)
+    )
+    (property "Datasheet" "~" (id 3) (at 243.84 151.13 0)
+      (effects (font (size 1.27 1.27)) hide)
+    )
+    (pin "1")
+  )
+  (symbol (lib_id "Mechanical:MountingHole_Pad") (at 259.08 151.13 0) (unit 1)
+    (in_bom yes) (on_board yes)
+    (property "Reference" "H4" (id 0) (at 257.81 146.05 0)
+      (effects (font (size 1.27 1.27)) (justify left))
+    )
+    (property "Value" "MountingHole_Pad" (id 1) (at 261.62 151.5622 0)
+      (effects (font (size 1.27 1.27)) (justify left) hide)
+    )
+    (property "Footprint" "MountingHole:MountingHole_2.2mm_M2_DIN965_Pad" (id 2) (at 259.08 151.13 0)
+      (effects (font (size 1.27 1.27)) hide)
+    )
+    (property "Datasheet" "~" (id 3) (at 259.08 151.13 0)
+      (effects (font (size 1.27 1.27)) hide)
+    )
+    (pin "1")
+  )
+  (symbol (lib_id "Mechanical:MountingHole_Pad") (at 248.92 151.13 0) (unit 1)
+    (in_bom yes) (on_board yes)
+    (property "Reference" "H2" (id 0) (at 247.65 146.05 0)
+      (effects (font (size 1.27 1.27)) (justify left))
+    )
+    (property "Value" "MountingHole_Pad" (id 1) (at 251.46 151.5622 0)
+      (effects (font (size 1.27 1.27)) (justify left) hide)
+    )
+    (property "Footprint" "MountingHole:MountingHole_2.2mm_M2_DIN965_Pad" (id 2) (at 248.92 151.13 0)
+      (effects (font (size 1.27 1.27)) hide)
+    )
+    (property "Datasheet" "~" (id 3) (at 248.92 151.13 0)
+      (effects (font (size 1.27 1.27)) hide)
+    )
+    (pin "1")
+  )
   (symbol (lib_id "power:+3.3V") (at 257.81 25.4 0) (unit 1)
     (in_bom yes) (on_board yes) (fields_autoplaced)
@@
     )
     (property "Datasheet" "" (id 3) (at 257.81 25.4 0)
+      (effects (font (size 1.27 1.27)) hide)
+    )
+    (pin "1")
+  )
+  (symbol (lib_id "power:GND") (at 251.46 158.75 0) (unit 1)
+    (in_bom yes) (on_board yes)
+    (property "Reference" "#PWR01" (id 0) (at 251.46 165.1 0)
+      (effects (font (size 1.27 1.27)) hide)
+    )
+    (property "Value" "GND" (id 1) (at 251.587 163.1442 0))
+    (property "Footprint" "" (id 2) (at 251.46 158.75 0)
+      (effects (font (size 1.27 1.27)) hide)
+    )
+    (property "Datasheet" "" (id 3) (at 251.46 158.75 0)
       (effects (font (size 1.27 1.27)) hide)
     )
@@
       (reference "#FLG0101") (unit 1) (value "PWR_FLAG") (footprint "")
     )
+    (path "/fc7091d6-82e4-43ad-bbf2-a8425e1bc812"
+      (reference "#PWR01") (unit 1) (value "GND") (footprint "")
+    )
     (path "/00000000-0000-0000-0000-000060e78127"
       (reference "#PWR02") (unit 1) (value "+5V") (footprint "")
@@
       (reference "D3") (unit 1) (value "GREEN") (footprint "LED_SMD:LED_0805_2012Metric_Pad1.15x1.40mm_HandSolder")
     )
+    (path "/83d65180-8fe4-4971-8e64-df9b48927213"
+      (reference "H1") (unit 1) (value "MountingHole_Pad") (footprint "MountingHole:MountingHole_2.2mm_M2_DIN965_Pad")
+    )
+    (path "/c2782eb1-3937-4cfb-8f6a-2e58f489cc50"
+      (reference "H2") (unit 1) (value "MountingHole_Pad") (footprint "MountingHole:MountingHole_2.2mm_M2_DIN965_Pad")
+    )
+    (path "/2282482a-d72f-4f6c-bde0-18bf1a7454bc"
+      (reference "H3") (unit 1) (value "MountingHole_Pad") (footprint "MountingHole:MountingHole_2.2mm_M2_DIN965_Pad")
+    )
+    (path "/94daf55a-df14-47e3-8c1f-72b1d555162a"
+      (reference "H4") (unit 1) (value "MountingHole_Pad") (footprint "MountingHole:MountingHole_2.2mm_M2_DIN965_Pad")
+    )
     (path "/00000000-0000-0000-0000-000060ddcbd6"
